File: kicad/mcu_n_tft.kicad_sch (KiCad schematic)
At the start: 14 parts, among them Q3 SS8050-G, Q4 SS8050-G, SW1 SW_MEC_5G, SW2 SW_MEC_5G, U4 ESP32-S3-Rx

Commit message: remove Rx with 0 Ohms
Parts:
- removed R33: 0R, Resistor_SMD:R_0603_1608Metric, symbol Device:R
Connections:
- net +3V3: now also U4.2 (3V3)
- net SPICLK: now also U4.11 (IO18); no longer U4.9 (IO16)
- net SPICS0: now also U4.8 (IO15); no longer U4.10 (IO17)
- net SPID: now also U4.10 (IO17); no longer U4.11 (IO18)
- net SPIQ: now also U4.9 (IO16); no longer U4.13 (IO19)
- net ~{INT}: now also U4.13 (IO19); no longer U4.14 (IO20)
- net ~{PD}: now also U4.14 (IO20); no longer U4.8 (IO15)
- no-connect marks 13 -> 9
Changed lines of the file:
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@@
   (no_connect (at 213.36 124.46))
   (no_connect (at 213.36 109.22))
-  (no_connect (at 213.36 111.76))
-  (no_connect (at 213.36 114.3))
-  (no_connect (at 213.36 116.84))
-  (no_connect (at 213.36 119.38))
   (no_connect (at 213.36 121.92))
   (no_connect (at 180.34 67.31))
@@
     (stroke (width 0) (type default) (color 0 0 0 0))
   )
+  (wire (pts (xy 213.36 111.76) (xy 220.98 111.76))
+    (stroke (width 0) (type default) (color 0 0 0 0))
+  )
   (wire (pts (xy 180.34 76.2) (xy 172.72 76.2))
     (stroke (width 0) (type default) (color 0 0 0 0))
@@
     (stroke (width 0) (type default) (color 0 0 0 0))
   )
+  (wire (pts (xy 213.36 119.38) (xy 220.98 119.38))
+    (stroke (width 0) (type default) (color 0 0 0 0))
+  )
   (wire (pts (xy 199.39 138.43) (xy 196.85 138.43))
     (stroke (width 0) (type default) (color 0 0 0 0))
@@
     (stroke (width 0) (type default) (color 0 0 0 0))
   )
+  (wire (pts (xy 213.36 114.3) (xy 220.98 114.3))
+    (stroke (width 0) (type default) (color 0 0 0 0))
+  )
   (wire (pts (xy 199.39 135.89) (xy 199.39 138.43))
     (stroke (width 0) (type default) (color 0 0 0 0))
@@
     (stroke (width 0) (type default) (color 0 0 0 0))
   )
-  (wire (pts (xy 172.72 43.18) (xy 172.72 53.34))
+  (wire (pts (xy 172.72 38.1) (xy 172.72 53.34))
     (stroke (width 0) (type default) (color 0 0 0 0))
   )
@@
     (stroke (width 0) (type default) (color 0 0 0 0))
   )
-  (wire (pts (xy 172.72 30.48) (xy 172.72 35.56))
-    (stroke (width 0) (type default) (color 0 0 0 0))
-  )
   (wire (pts (xy 158.75 45.72) (xy 158.75 43.18))
     (stroke (width 0) (type default) (color 0 0 0 0))
@@
   )
   (wire (pts (xy 109.22 45.72) (xy 116.84 45.72))
+    (stroke (width 0) (type default) (color 0 0 0 0))
+  )
+  (wire (pts (xy 213.36 116.84) (xy 220.98 116.84))
     (stroke (width 0) (type default) (color 0 0 0 0))
   )
@@
     (effects (font (size 1.27 1.27)) (justify left))
   )
-  (hierarchical_label "SPICLK" (shape output) (at 220.98 93.98 0)
-    (effects (font (size 1.27 1.27)) (justify left))
-  )
-  (hierarchical_label "~{PD}" (shape output) (at 220.98 91.44 0)
-    (effects (font (size 1.27 1.27)) (justify left))
-  )
-  (hierarchical_label "SPID" (shape output) (at 220.98 99.06 0)
-    (effects (font (size 1.27 1.27)) (justify left))
-  )
-  (hierarchical_label "SPIQ" (shape output) (at 220.98 101.6 0)
-    (effects (font (size 1.27 1.27)) (justify left))
-  )
-  (hierarchical_label "SPICS0" (shape output) (at 220.98 96.52 0)
+  (hierarchical_label "SPICLK" (shape output) (at 220.98 99.06 0)
+    (effects (font (size 1.27 1.27)) (justify left))
+  )
+  (hierarchical_label "~{PD}" (shape output) (at 220.98 104.14 0)
+    (effects (font (size 1.27 1.27)) (justify left))
+  )
+  (hierarchical_label "SPID" (shape output) (at 220.98 96.52 0)
+    (effects (font (size 1.27 1.27)) (justify left))
+  )
+  (hierarchical_label "SPIQ" (shape output) (at 220.98 93.98 0)
+    (effects (font (size 1.27 1.27)) (justify left))
+  )
+  (hierarchical_label "SPICS0" (shape output) (at 220.98 91.44 0)
     (effects (font (size 1.27 1.27)) (justify left))
   )
@@
     (effects (font (size 1.27 1.27)) (justify left))
   )
-  (hierarchical_label "~{INT}" (shape input) (at 220.98 104.14 0)
+  (hierarchical_label "~{INT}" (shape input) (at 220.98 101.6 0)
     (effects (font (size 1.27 1.27)) (justify left))
   )
@@
     (pin "2")
   )
-  (symbol (lib_id "Device:R") (at 172.72 39.37 180) (unit 1)
-    (in_bom yes) (on_board yes)
-    (property "Reference" "R33" (id 0) (at 170.18 39.37 90))
-    (property "Value" "0R" (id 1) (at 175.26 39.37 90))
-    (property "Footprint" "Resistor_SMD:R_0603_1608Metric" (id 2) (at 174.498 39.37 90)
-      (effects (font (size 1.27 1.27)) hide)
-    )
-    (property "Datasheet" "~" (id 3) (at 172.72 39.37 0)
-      (effects (font (size 1.27 1.27)) hide)
-    )
-    (property "Digikey" "541-0.0SBCT-ND" (id 4) (at 172.72 39.37 0)
-      (effects (font (size 1.27 1.27)) hide)
-    )
-    (pin "1")
-    (pin "2")
-  )
   (symbol (lib_id "Device:R") (at 105.41 45.72 270) (unit 1)
     (in_bom yes) (on_board yes)
@@
     (pin "2")
   )
-  (symbol (lib_id "power:+3V3") (at 172.72 30.48 0) (unit 1)
-    (in_bom yes) (on_board yes)
-    (property "Reference" "#PWR053" (id 0) (at 172.72 34.29 0)
-      (effects (font (size 1.27 1.27)) hide)
-    )
-    (property "Value" "+3V3" (id 1) (at 173.101 26.0858 0))
-    (property "Footprint" "" (id 2) (at 172.72 30.48 0)
-      (effects (font (size 1.27 1.27)) hide)
-    )
-    (property "Datasheet" "" (id 3) (at 172.72 30.48 0)
-      (effects (font (size 1.27 1.27)) hide)
-    )
+  (symbol (lib_id "power:+3V3") (at 172.72 38.1 0) (unit 1)
+    (in_bom yes) (on_board yes)
+    (property "Reference" "#PWR053" (id 0) (at 172.72 41.91 0)
+      (effects (font (size 1.27 1.27)) hide)
+    )
+    (property "Value" "+3V3" (id 1) (at 173.101 33.7058 0))
+    (property "Footprint" "" (id 2) (at 172.72 38.1 0)
+      (effects (font (size 1.27 1.27)) hide)
+    )
+    (property "Datasheet" "" (id 3) (at 172.72 38.1 0)
+      (effects (font (size 1.27 1.27)) hide)
+    )
