File: kicad/usb_uart.kicad_sch (KiCad schematic)
At the start: 11 parts, among them Q5 DMN2004WK-7, U5 CP2102N-Axx-xQFN28

Commit message: remove Rx with 0 Ohms
Parts:
- removed R38, R39: 0R, Resistor_SMD:R_0603_1608Metric, symbol Device:R
Connections:
- net CHREN_: now also Q5.1 (G), R40.2
- no-connect marks 13 -> 14
Changed lines of the file:
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@@
   (no_connect (at 134.62 120.65))
   (no_connect (at 134.62 118.11))
+  (no_connect (at 121.92 69.85))
   (no_connect (at 134.62 110.49))
   (no_connect (at 134.62 92.71))
@@
     (stroke (width 0) (type default) (color 0 0 0 0))
   )
-  (wire (pts (xy 119.38 55.88) (xy 119.38 69.85))
+  (wire (pts (xy 119.38 62.23) (xy 119.38 69.85))
     (stroke (width 0) (type default) (color 0 0 0 0))
   )
@@
     (stroke (width 0) (type default) (color 0 0 0 0))
   )
-  (wire (pts (xy 179.07 93.98) (xy 189.23 93.98))
-    (stroke (width 0) (type default) (color 0 0 0 0))
-  )
   (wire (pts (xy 154.94 68.58) (xy 154.94 69.85))
     (stroke (width 0) (type default) (color 0 0 0 0))
@@
     (stroke (width 0) (type default) (color 0 0 0 0))
   )
-  (wire (pts (xy 121.92 69.85) (xy 121.92 67.31))
-    (stroke (width 0) (type default) (color 0 0 0 0))
-  )
-  (wire (pts (xy 129.54 55.88) (xy 129.54 58.42))
-    (stroke (width 0) (type default) (color 0 0 0 0))
-  )
   (wire (pts (xy 121.92 135.89) (xy 121.92 139.7))
     (stroke (width 0) (type default) (color 0 0 0 0))
@@
     (stroke (width 0) (type default) (color 0 0 0 0))
   )
-  (wire (pts (xy 129.54 66.04) (xy 129.54 67.31))
-    (stroke (width 0) (type default) (color 0 0 0 0))
-  )
   (wire (pts (xy 215.9 85.09) (xy 223.52 85.09))
     (stroke (width 0) (type default) (color 0 0 0 0))
@@
     (stroke (width 0) (type default) (color 0 0 0 0))
   )
-  (wire (pts (xy 196.85 93.98) (xy 205.74 93.98))
-    (stroke (width 0) (type default) (color 0 0 0 0))
-  )
-  (wire (pts (xy 121.92 67.31) (xy 129.54 67.31))
+  (wire (pts (xy 195.58 93.98) (xy 205.74 93.98))
     (stroke (width 0) (type default) (color 0 0 0 0))
   )
@@
     (effects (font (size 1.27 1.27)) (justify right bottom))
   )
-  (label "CHREN_" (at 179.07 93.98 0)
+  (label "CHREN_" (at 195.58 93.98 0)
     (effects (font (size 1.27 1.27)) (justify left bottom))
   )
@@
     (pin "1")
   )
-  (symbol (lib_id "Device:R") (at 129.54 62.23 0) (unit 1)
-    (in_bom yes) (on_board yes)
-    (property "Reference" "R38" (id 0) (at 127 62.23 90))
-    (property "Value" "0R" (id 1) (at 132.08 62.23 90))
-    (property "Footprint" "Resistor_SMD:R_0603_1608Metric" (id 2) (at 127.762 62.23 90)
-      (effects (font (size 1.27 1.27)) hide)
-    )
-    (property "Datasheet" "~" (id 3) (at 129.54 62.23 0)
-      (effects (font (size 1.27 1.27)) hide)
-    )
-    (property "Digikey" "541-0.0SBCT-ND" (id 4) (at 129.54 62.23 0)
-      (effects (font (size 1.27 1.27)) hide)
-    )
-    (pin "1")
-    (pin "2")
-  )
   (symbol (lib_id "power:GND") (at 205.74 106.68 0) (unit 1)
     (in_bom yes) (on_board yes)
@@
     (pin "2")
   )
-  (symbol (lib_id "power:+3V3") (at 129.54 55.88 0) (unit 1)
-    (in_bom yes) (on_board yes)
-    (property "Reference" "#PWR063" (id 0) (at 129.54 59.69 0)
-      (effects (font (size 1.27 1.27)) hide)
-    )
-    (property "Value" "+3V3" (id 1) (at 129.54 52.07 0))
-    (property "Footprint" "" (id 2) (at 129.54 55.88 0)
-      (effects (font (size 1.27 1.27)) hide)
-    )
-    (property "Datasheet" "" (id 3) (at 129.54 55.88 0)
-      (effects (font (size 1.27 1.27)) hide)
-    )
-    (pin "1")
-  )
-  (symbol (lib_id "power:VAA") (at 119.38 55.88 0) (unit 1)
-    (in_bom yes) (on_board yes)
-    (property "Reference" "#PWR061" (id 0) (at 119.38 59.69 0)
-      (effects (font (size 1.27 1.27)) hide)
-    )
-    (property "Value" "VAA" (id 1) (at 119.38 52.07 0))
-    (property "Footprint" "" (id 2) (at 119.38 55.88 0)
-      (effects (font (size 1.27 1.27)) hide)
-    )
-    (property "Datasheet" "" (id 3) (at 119.38 55.88 0)
-      (effects (font (size 1.27 1.27)) hide)
-    )
-    (pin "1")
-  )
-  (symbol (lib_id "Device:R") (at 193.04 93.98 270) (unit 1)
-    (in_bom yes) (on_board yes)
-    (property "Reference" "R39" (id 0) (at 193.04 91.44 90))
-    (property "Value" "0R" (id 1) (at 193.04 96.52 90))
-    (property "Footprint" "Resistor_SMD:R_0603_1608Metric" (id 2) (at 193.04 92.202 90)
-      (effects (font (size 1.27 1.27)) hide)
-    )
-    (property "Datasheet" "~" (id 3) (at 193.04 93.98 0)
-      (effects (font (size 1.27 1.27)) hide)
-    )
-    (property "Digikey" "541-0.0SBCT-ND" (id 4) (at 193.04 93.98 0)
-      (effects (font (size 1.27 1.27)) hide)
-    )
-    (pin "1")
-    (pin "2")
+  (symbol (lib_id "power:VAA") (at 119.38 62.23 0) (unit 1)
+    (in_bom yes) (on_board yes)
+    (property "Reference" "#PWR061" (id 0) (at 119.38 66.04 0)
+      (effects (font (size 1.27 1.27)) hide)
+    )
+    (property "Value" "VAA" (id 1) (at 119.38 58.42 0))
+    (property "Footprint" "" (id 2) (at 119.38 62.23 0)
+      (effects (font (size 1.27 1.27)) hide)
+    )
+    (property "Datasheet" "" (id 3) (at 119.38 62.23 0)
+      (effects (font (size 1.27 1.27)) hide)
+    )
+    (pin "1")
   )
   (symbol (lib_id "power:GND") (at 121.92 139.7 0) (unit 1)
